File: CH4D3M0 Rev 1.brd (EAGLE design)
At the start: 85.6 x 54 mm, 55 parts, among them T7 2N2222, T8 2N2222, U1 ANALOG_DEVICES_INC_ADM3052ANA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

Commit message: Add files via upload
Parts:
- added D1: (no value), diode:D-5
- C20, C22: value 10 nF -> 10 uF
- moved D3 6.77 mm to (57.3, 18.0), turned to 0 degrees
- moved LED1 4.99 mm to (76.8, 14.5), turned to 270 degrees
- moved R11 4.98 mm to (68.2, 16.8), turned to 90 degrees
- moved R13 4.80 mm to (61.6, 14.9)
- moved R12 4.10 mm to (61.7, 11.7)
- moved LED2 3.61 mm to (76.8, 10.4)
- moved T2 2.97 mm to (57.5, 22.3), turned to 180 degrees
- moved R9 2.55 mm to (73.7, 27.1)
- moved R8 2.01 mm to (66.1, 30.2)
- moved R17 1.39 mm to (62.9, 30.2)
- moved C22 1.05 mm to (48.0, 34.1)
- moved R15 1.02 mm to (78.1, 33.4)
- moved R16 0.80 mm to (59.8, 30.2)
Connections:
- net N$11: now also D1.C
- net N$15: now also D1.A
Routing:
- net GND: track 302.1 -> 279.3 mm
- net N$34: track 49.4 -> 36.5 mm
- net N$19: track 80.0 -> 68.6 mm
- net N$1: track 79.3 -> 68.6 mm
- net +3V3: track 85.0 -> 75.1 mm
- net N$21: track 65.0 -> 55.6 mm
- net N$26: track 9.61 -> 2.58 mm
- net N$23: track 75.6 -> 71.3 mm
- net N$33: track 4.07 -> 7.89 mm
- net N$11: track 81.0 -> 83.9 mm
- net N$30: track 40.6 -> 37.8 mm
- net N$32: track 9.15 -> 6.88 mm
- net N$6: track 27.7 -> 29.7 mm
- net N$15: track 26.4 -> 28.3 mm
- net N$12: track 25.1 -> 27.0 mm
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Other:
- board text added: "CH4D3M0 Shield V1.1"
- board text removed: "CH4D3M0 Shield V1.0"
